File: PCB/Epoch-Mainboard/Epoch-Mainboard.kicad_sch (KiCad schematic)
At the start: 48 parts, among them J1 USB_C_Receptacle_PowerOnly_6P, J2 Conn_02x06_Odd_Even, J3 Conn_02x06_Odd_Even, SW1 SW_SPDT, U1 PCA9685PW, U2 MCP73831-4-OT

Commit message: Part value changes.
Parts:
- R10: value ??? -> 2K
- R12: value 2K -> 1K
- U2: value MCP73831-4-OT -> MCP73831T-2ACI/OT
Changed lines of the file:
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@@
 			)
 		)
-		(property "Value" "???"
+		(property "Value" "2K"
 			(at 118.11 133.604 90)
 			(effects
@@
 			)
 		)
-		(property "Value" "MCP73831-4-OT"
+		(property "Value" "MCP73831T-2ACI/OT"
 			(at 122.936 127 0)
 			(effects
 				(font
-					(size 1 1)
+					(size 0.8 0.8)
 					(thickness 0.2)
 					(bold yes)
@@
 			)
 		)
-		(property "Value" "2K"
+		(property "Value" "1K"
 			(at 140.97 141.224 90)
 			(effects
